Commit message: URDF bugfixes

File: youbot_description/urdf/youbot_arm/arm.transmission.xacro (robot description, xacro)
@@ -7,16 +7,16 @@
 	<!-- reduction ratio must not to be 0-->
 	<xacro:macro name="youbot_arm_transmission" params="name">
-		<transmission name="${name}_trans_1">
-      <type>transmission_interface/SimpleTransmission</type>
-			<actuator name="${name}_motor_1">
-        <hardwareInterface>EffortJointInterface</hardwareInterface>
-        <mechanicalReduction>1</mechanicalReduction>
-      </actuator>
-			<joint name="${name}_joint_1">
-        <hardwareInterface>EffortJointInterface</hardwareInterface>
-      </joint>
-		</transmission>
-		<transmission name="${name}_trans_2">
-      <type>transmission_interface/SimpleTransmission</type>
+	<transmission name="${name}_trans_1">
+      		<type>transmission_interface/SimpleTransmission</type>
+		<actuator name="${name}_motor_1">
+        		<hardwareInterface>EffortJointInterface</hardwareInterface>
+        		<mechanicalReduction>1</mechanicalReduction>
+      		</actuator>
+		<joint name="${name}_joint_1">
+        		<hardwareInterface>EffortJointInterface</hardwareInterface>
+      		</joint>
+	</transmission>
+	<transmission name="${name}_trans_2">
+      	<type>transmission_interface/SimpleTransmission</type>
 			<actuator name="${name}_motor_2">
         <hardwareInterface>EffortJointInterface</hardwareInterface>

File: youbot_description/urdf/youbot_arm/arm.urdf.xacro (robot description, xacro)
@@ -10,5 +10,5 @@
 		<!-- joint between base_link and arm_0_link -->
 		<joint name="${name}_joint_0" type="fixed" >
-			<insert_block name="origin" />
+			<xacro:insert_block name="origin" />
 			<parent link="${parent}" />
 			<child link="${name}_link_0" />
@@ -44,11 +44,11 @@
 			<axis xyz="0 0 -1"/>
 			<!--<calibration rising="${arm_1_ref}" falling="${arm_1_ref}"/>-->
-			<dynamics damping="1" friction="1" />
+			<dynamics damping="0" friction="0" />
 			<!-- damping - N*s/m, N*s*m/rad -->
 			<!-- friction - N, N*m -->
-			<limit effort="${9.5}" velocity="${M_PI / 2.0}" lower="0" upper="${joint_1_limit}"/>
+			<limit effort="${9.5}" velocity="${M_PI/2}" lower="0" upper="${joint_1_limit}"/>
 			<!--effort - N, N*m-->
 			<!--velocity - m/s, rad/s-->
-			<safety_controller k_position="20" k_velocity="${9.5/M_PI / 2.0}" soft_lower_limit="${threshold}" soft_upper_limit="${joint_1_limit_soft}" />
+                        <!--safety_controller k_position="20" k_velocity="${9.5/M_PI / 2.0}" soft_lower_limit="${threshold}" soft_upper_limit="${joint_1_limit_soft}" /-->
 			<!--k_position N/m, N/rad-->
 			<!--k_velocity N*s/m, N*s*m/rad-->
