Commit message: added asus xtion camera to youbot gripper and fixed a lot of warnings and bugs

File: youbot_description/robots/youbot.urdf.xacro (robot description, xacro)
@@ -22,4 +22,5 @@
   <!-- sensors -->
   <xacro:include filename="$(find youbot_description)/urdf/sensors/hokuyo_urg04_laser.urdf.xacro"/>
+  <xacro:include filename="$(find youbot_description)/urdf/sensors/asus_xtion_camera.urdf.xacro"/>
   <!-- Now we can start using the macros xacro:included above to define the actual youbot -->
   <!-- The first use of a macro.  This one was defined in base.urdf.xacro above.
@@ -42,6 +43,11 @@
   </xacro:youbot_gripper>
   <!-- base laser front -->
-  <xacro:hokuyo_urg04_laser name="base_laser_front" parent="base" ros_topic="base_scan" update_rate="10" min_angle="-1.57" max_angle="1.57">
+ <!-- <xacro:macro name="hokuyo_urg04_laser" params="name parent *origin ros_topic update_rate min_angle max_angle"> -->
+  <xacro:hokuyo_urg04_laser name="base_laser_front" parent="base" ros_topic="scan" update_rate="10" min_angle="-1.57" max_angle="1.57">
     <origin xyz="0.3 0 -0.03" rpy="0 0 0"/>
   </xacro:hokuyo_urg04_laser>
+ <!-- <xacro:macro name="asus_xtion_camera" params="name parent *origin tilt"> -->
+  <xacro:asus_xtion_camera name="xtion" parent="gripper_palm_link" tilt="0">
+    <origin xyz="0 0 0" rpy="0 -1.57 0"/>
+  </xacro:asus_xtion_camera>
 </robot>

File: youbot_description/urdf/sensors/asus_xtion_camera.gazebo.xacro (robot description, xacro)
@@ -1,7 +1,8 @@
 <?xml version="1.0"?>
-<root xmlns:sensor="http://playerstage.sourceforge.net/gazebo/xmlschema/#sensor"
+<root xmlns:xacro="http://ros.org/wiki/xacro">
+  <!--xmlns:interface="http://playerstage.sourceforge.net/gazebo/xmlschema/#interface"
+      xmlns:sensor="http://playerstage.sourceforge.net/gazebo/xmlschema/#sensor"
       xmlns:controller="http://playerstage.sourceforge.net/gazebo/xmlschema/#controller"
-      xmlns:interface="http://playerstage.sourceforge.net/gazebo/xmlschema/#interface"
-      xmlns:xacro="http://ros.org/wiki/xacro">
+  -->
 <xacro:macro name="asus_xtion_camera_gazebo" params="name">
   <xacro:asus_xtion_depth_camera_gazebo name="${name}" />
@@ -10,55 +11,82 @@
 <xacro:macro name="asus_xtion_depth_camera_gazebo" params="name">
   <gazebo reference="${name}_depth_frame">
-    <sensor:camera name="${name}_depth_frame_sensor">
-      <imageFormat>R8G8B8</imageFormat>
-      <imageSize>640 480</imageSize>
-      <hfov>57</hfov>
-      <nearClip>0.01</nearClip>
-      <farClip>5</farClip>
-      <updateRate>20.0</updateRate>
-      <baseline>0.2</baseline>
-      <controller:gazebo_ros_camera name="${name}_depth_frame_controller" plugin="libgazebo_ros_camera.so">
+    <sensor name="${name}_depth" type="camera">
+      <update_rate>30.0</update_rate>
+      <camera name="gripper_depth_cam">
+        <horizontal_fov>1.3962634</horizontal_fov>
+        <image>
+          <width>640</width>
+          <height>480</height>
+          <format>R8G8B8</format>
+        </image>
+        <clip>
+          <near>0.02</near>
+          <far>300</far>
+        </clip>
+        <noise>
+          <type>gaussian</type>
+          <!-- Noise is sampled independently per pixel on each frame.
+               That pixel's noise value is added to each of its color
+               channels, which at that point lie in the range [0,1]. -->
+          <mean>0.0</mean>
+          <stddev>0.007</stddev>
+        </noise>
+      </camera>
+      <plugin name="camera_controller" filename="libgazebo_ros_camera.so">
         <alwaysOn>true</alwaysOn>
         <updateRate>20.0</updateRate>
-        <imageTopicName>/camera/ir/image_raw</imageTopicName>
-        <cameraInfoTopicName>/camera/ir/camera_info</cameraInfoTopicName>
-        <depthImageTopicName>/camera/depth/image_raw</depthImageTopicName>
-        <depthImageInfoTopicName>/camera/depth/camera_info</depthImageInfoTopicName>
-        <pointCloudTopicName>/camera/depth/points</pointCloudTopicName>
-        <frameName>/${name}_depth_optical_frame</frameName>
-        <pointCloudCutoff>0.5</pointCloudCutoff>
-        <distortion_k1>0.00000001</distortion_k1>
-        <distortion_k2>0.00000001</distortion_k2>
-        <distortion_k3>0.00000001</distortion_k3>
-        <distortion_t1>0.00000001</distortion_t1>
-        <distortion_t2>0.00000001</distortion_t2>
-      </controller:gazebo_ros_camera>
-    </sensor:camera>
-  </gazebo>
+        <cameraName>camera/depth</cameraName>
+        <imageTopicName>image_raw</imageTopicName>
+        <cameraInfoTopicName>camera_info</cameraInfoTopicName>
+        <frameName>${name}_depth_frame</frameName>
+        <hackBaseline>0.07</hackBaseline>
+        <distortionK1>0.0</distortionK1>
+        <distortionK2>0.0</distortionK2>
+        <distortionK3>0.0</distortionK3>
+        <distortionT1>0.0</distortionT1>
+        <distortionT2>0.0</distortionT2>
+      </plugin>
+    </sensor>
+</gazebo>
 </xacro:macro>
 <xacro:macro name="asus_xtion_rgb_camera_gazebo" params="name">
   <gazebo reference="${name}_rgb_frame">
-    <sensor:camera name="${name}_rgb_frame_sensor">
-      <imageFormat>R8G8B8</imageFormat>
-      <imageSize>640 480</imageSize>
-      <hfov>57</hfov>
-      <nearClip>0.01</nearClip>
-      <farClip>5</farClip>
-      <updateRate>20.0</updateRate>
-      <baseline>0.2</baseline>
-      <controller:gazebo_ros_camera name="${name}_rgb_frame_controller" plugin="libgazebo_ros_camera.so">
+    <sensor name="${name}_rgb" type="camera">
+      <update_rate>30.0</update_rate>
+      <camera name="gripper_rgb_cam">
+        <horizontal_fov>1.3962634</horizontal_fov>
+        <image>
+          <width>640</width>
+          <height>480</height>
+          <format>R8G8B8</format>
+        </image>
+	<clip>
+          <near>0.02</near>
+          <far>300</far>
+        </clip>
+        <noise>
+          <type>gaussian</type>
+          <!-- Noise is sampled independently per pixel on each frame.
+               That pixel's noise value is added to each of its color
+               channels, which at that point lie in the range [0,1]. -->
+          <mean>0.0</mean>
+          <stddev>0.007</stddev>
+        </noise>
+      </camera>
+      <plugin name="camera_controller" filename="libgazebo_ros_camera.so">
         <alwaysOn>true</alwaysOn>
         <updateRate>20.0</updateRate>
-        <imageTopicName>/camera/rgb/image_raw</imageTopicName>
-        <cameraInfoTopicName>/camera/rgb/camera_info</cameraInfoTopicName>
-        <frameName>/${name}_rgb_optical_frame</frameName>
-        <pointCloudCutoff>0.5</pointCloudCutoff>
-        <distortion_k1>0.00000001</distortion_k1>
-        <distortion_k2>0.00000001</distortion_k2>
-        <distortion_k3>0.00000001</distortion_k3>
-        <distortion_t1>0.00000001</distortion_t1>
-        <distortion_t2>0.00000001</distortion_t2>
-      </controller:gazebo_ros_camera>
-    </sensor:camera>
+        <cameraName>camera/rgb</cameraName>
+        <imageTopicName>image_raw</imageTopicName>
+        <cameraInfoTopicName>camera_info</cameraInfoTopicName>
+        <frameName>${name}_rgb_frame</frameName>
+        <hackBaseline>0.07</hackBaseline>
+        <distortionK1>0.0</distortionK1>
+        <distortionK2>0.0</distortionK2>
+        <distortionK3>0.0</distortionK3>
+        <distortionT1>0.0</distortionT1>
+        <distortionT2>0.0</distortionT2>
+      </plugin>
+    </sensor>
   </gazebo>
 </xacro:macro>

File: youbot_description/urdf/sensors/asus_xtion_camera.urdf.xacro (robot description, xacro)
@@ -1,4 +1,4 @@
 <?xml version="1.0"?>
-<root xmlns:xacro="http://playerstage.sourceforge.net/gazebo/xmlschema/#interface">
+<root xmlns:xacro="http://ros.org/wiki/xacro">
   <xacro:include filename="$(find youbot_description)/urdf/sensors/asus_xtion_camera.gazebo.xacro" />
   <xacro:property name="eye_x_offset" value="0.03" />

File: youbot_description/urdf/sensors/hokuyo_urg04_laser.gazebo.xacro (robot description, xacro)
@@ -7,30 +7,30 @@
     <gazebo reference="${name}_link">
       <sensor name="${name}" type="ray">
-		<always_on>true</always_on>
+	<always_on>true</always_on>
         <update_rate>${update_rate}</update_rate>
-		<pose>0 0 0 0 0 0</pose>
-		<visualize>false</visualize>
+	<pose>0 0 0 0 0 0</pose>
+	<visualize>false</visualize>
         <ray>
-            <scan>
-                <horizontal>
-                    <samples>150</samples>
-                    <resolution>1.0</resolution>
-                    <min_angle>${min_angle}</min_angle>
-                    <max_angle>${max_angle}</max_angle>
-                </horizontal>
-            </scan>
-            <range>
-				<min>0.05</min>
-				<max>5.6</max>
-				<resolution>0.36</resolution>
-			</range>
+          <scan>
+            <horizontal>
+              <samples>150</samples>
+              <resolution>1.0</resolution>
+              <min_angle>${min_angle}</min_angle>
+              <max_angle>${max_angle}</max_angle>
+            </horizontal>
+          </scan>
+          <range>
+	    <min>0.05</min>
+	    <max>5.6</max>
+	    <resolution>0.36</resolution>
+	  </range>
         </ray>
         <plugin name="gazebo_ros_${name}_controller" filename="libgazebo_ros_laser.so">
-            <gaussianNoise>0.005</gaussianNoise>
-            <alwaysOn>true</alwaysOn>
-            <updateRate>${update_rate}</updateRate>
-            <topicName>${ros_topic}</topicName>
-            <frameName>/${name}_link</frameName>
-         </plugin>
+          <gaussianNoise>0.005</gaussianNoise>
+          <alwaysOn>true</alwaysOn>
+          <updateRate>${update_rate}</updateRate>
+          <topicName>${ros_topic}</topicName>
+          <frameName>/${name}_link</frameName>
+        </plugin>
       </sensor>
     </gazebo>

Commit message: changed effort controller to position controller and changed position of asus xtion camera in URDF

File: youbot_description/robots/youbot.urdf.xacro (robot description, xacro)
@@ -49,5 +49,5 @@
  <!-- <xacro:macro name="asus_xtion_camera" params="name parent *origin tilt"> -->
   <xacro:asus_xtion_camera name="xtion" parent="gripper_palm_link" tilt="0">
-    <origin xyz="0 0 0" rpy="0 -1.57 0"/>
+    <origin xyz="0 0 0" rpy="3.14159 -1.57 0"/>
   </xacro:asus_xtion_camera>
 </robot>

File: youbot_description/urdf/youbot_arm/arm.transmission.xacro (robot description, xacro)
@@ -10,9 +10,9 @@
       		<type>transmission_interface/SimpleTransmission</type>
 		<actuator name="${name}_motor_1">
-        		<hardwareInterface>hardware_interface/EffortJointInterface</hardwareInterface>
+        		<hardwareInterface>hardware_interface/PositionJointInterface</hardwareInterface>
         		<mechanicalReduction>1</mechanicalReduction>
       		</actuator>
 		<joint name="${name}_joint_1">
-        		<hardwareInterface>hardware_interface/EffortJointInterface</hardwareInterface>
+        		<hardwareInterface>hardware_interface/PositionJointInterface</hardwareInterface>
       		</joint>
 	</transmission>
@@ -20,9 +20,9 @@
       	<type>transmission_interface/SimpleTransmission</type>
 			<actuator name="${name}_motor_2">
-        <hardwareInterface>hardware_interface/EffortJointInterface</hardwareInterface>
+        <hardwareInterface>hardware_interface/PositionJointInterface</hardwareInterface>
         <mechanicalReduction>1</mechanicalReduction>
       </actuator>
 			<joint name="${name}_joint_2">
-        <hardwareInterface>hardware_interface/EffortJointInterface</hardwareInterface>
+        <hardwareInterface>hardware_interface/PositionJointInterface</hardwareInterface>
       </joint>
 		</transmission>
@@ -30,9 +30,9 @@
       <type>transmission_interface/SimpleTransmission</type>
 			<actuator name="${name}_motor_3">
-        <hardwareInterface>hardware_interface/EffortJointInterface</hardwareInterface>
+        <hardwareInterface>hardware_interface/PositionJointInterface</hardwareInterface>
         <mechanicalReduction>1</mechanicalReduction>
       </actuator>
 			<joint name="${name}_joint_3">
-        <hardwareInterface>hardware_interface/EffortJointInterface</hardwareInterface>
+        <hardwareInterface>hardware_interface/PositionJointInterface</hardwareInterface>
       </joint>
 		</transmission>
@@ -40,9 +40,9 @@
       <type>transmission_interface/SimpleTransmission</type>
 			<actuator name="${name}_motor_4">
-        <hardwareInterface>hardware_interface/EffortJointInterface</hardwareInterface>
+        <hardwareInterface>hardware_interface/PositionJointInterface</hardwareInterface>
         <mechanicalReduction>1</mechanicalReduction>
       </actuator>
 			<joint name="${name}_joint_4">
-        <hardwareInterface>hardware_interface/EffortJointInterface</hardwareInterface>
+        <hardwareInterface>hardware_interface/PositionJointInterface</hardwareInterface>
       </joint>
 		</transmission>
@@ -50,9 +50,9 @@
       <type>transmission_interface/SimpleTransmission</type>
 			<actuator name="${name}_motor_5">
-        <hardwareInterface>hardware_interface/EffortJointInterface</hardwareInterface>
+        <hardwareInterface>hardware_interface/PositionJointInterface</hardwareInterface>
         <mechanicalReduction>1</mechanicalReduction>
       </actuator>
 			<joint name="${name}_joint_5">
-        <hardwareInterface>hardware_interface/EffortJointInterface</hardwareInterface>
+        <hardwareInterface>hardware_interface/PositionJointInterface</hardwareInterface>
       </joint>
 		</transmission>

File: youbot_description/urdf/youbot_gripper/gripper.transmission.xacro (robot description, xacro)
@@ -8,9 +8,9 @@
       <type>transmission_interface/SimpleTransmission</type>
 			<actuator name="${name}_finger_l_motor">
-        <hardwareInterface>hardware_interface/EffortJointInterface</hardwareInterface>
+        <hardwareInterface>hardware_interface/PositionJointInterface</hardwareInterface>
         <mechanicalReduction>1</mechanicalReduction>
       </actuator>
 			<joint name="${name}_finger_joint_l">
-        <hardwareInterface>hardware_interface/EffortJointInterface</hardwareInterface>
+        <hardwareInterface>hardware_interface/PositionJointInterface</hardwareInterface>
       </joint>
 		</transmission>
@@ -18,9 +18,9 @@
       <type>transmission_interface/SimpleTransmission</type>
 			<actuator name="${name}_finger_r_motor">
-        <hardwareInterface>hardware_interface/EffortJointInterface</hardwareInterface>
+        <hardwareInterface>hardware_interface/PositionJointInterface</hardwareInterface>
         <mechanicalReduction>1</mechanicalReduction>
       </actuator>
 			<joint name="${name}_finger_joint_r">
-        <hardwareInterface>hardware_interface/EffortJointInterface</hardwareInterface>
+        <hardwareInterface>hardware_interface/PositionJointInterface</hardwareInterface>
       </joint>
 		</transmission>
