Commit message: Changed Visual tag for wheels

File: youbot_description/urdf/youbot_base/base.urdf.xacro (robot description, xacro)
@@ -8,28 +8,28 @@
   <xacro:include filename="$(find youbot_description)/urdf/youbot_base/base.transmission.xacro"/>
   <!-- simplified box collision geometry for base -->
-  <xacro:property name="base_size_x" value="0.570"/>
-  <xacro:property name="base_size_y" value="0.360"/>
-  <xacro:property name="base_size_z" value="0.100"/>
-  <xacro:property name="base_mass" value="22.0"/>
-  <xacro:property name="caster_offset_x" value="0.228"/>
-  <xacro:property name="caster_offset_y" value="0.158"/>
-  <xacro:property name="caster_offset_z" value="-0.034"/>
-  <xacro:property name="caster_mass" value="0.1"/>
-  <xacro:property name="wheel_offset_x" value="0.0"/>
-  <xacro:property name="wheel_offset_y" value="0.0"/>
-  <xacro:property name="wheel_offset_z" value="0.0"/>
-  <xacro:property name="wheel_mass" value="0.4"/>
-  <xacro:property name="wheel_radius" value="0.05"/>
-  <xacro:property name="wheel_length" value="0.005"/>
-  <xacro:property name="caster_joint_damping" value="1.0"/>
-  <xacro:property name="caster_joint_friction" value="1.0"/>
-  <xacro:property name="caster_joint_effort" value="30"/>
-  <xacro:property name="caster_joint_velocity" value="10"/>
-  <xacro:property name="caster_joint_safety_k_velocity" value="10.0"/>
-  <xacro:property name="wheel_joint_damping" value="1.0"/>
-  <xacro:property name="wheel_joint_friction" value="1.0"/>
-  <xacro:property name="wheel_joint_effort" value="30"/>
-  <xacro:property name="wheel_joint_velocity" value="10"/>
-  <xacro:property name="wheel_joint_safety_k_velocity" value="10.0"/>
+  <property name="base_size_x" value="0.570"/>
+  <property name="base_size_y" value="0.360"/>
+  <property name="base_size_z" value="0.100"/>
+  <property name="base_mass" value="22.0"/>
+  <property name="caster_offset_x" value="0.228"/>
+  <property name="caster_offset_y" value="0.158"/>
+  <property name="caster_offset_z" value="-0.034"/>
+  <property name="caster_mass" value="0.1"/>
+  <property name="wheel_offset_x" value="0.0"/>
+  <property name="wheel_offset_y" value="0.0"/>
+  <property name="wheel_offset_z" value="0.0"/>
+  <property name="wheel_mass" value="0.4"/>
+  <property name="wheel_radius" value="0.05"/>
+  <property name="wheel_length" value="0.005"/>
+  <property name="caster_joint_damping" value="1.0"/>
+  <property name="caster_joint_friction" value="1.0"/>
+  <property name="caster_joint_effort" value="30"/>
+  <property name="caster_joint_velocity" value="10"/>
+  <property name="caster_joint_safety_k_velocity" value="10.0"/>
+  <property name="wheel_joint_damping" value="1.0"/>
+  <property name="wheel_joint_friction" value="1.0"/>
+  <property name="wheel_joint_effort" value="30"/>
+  <property name="wheel_joint_velocity" value="10"/>
+  <property name="wheel_joint_safety_k_velocity" value="10.0"/>
   <xacro:macro name="youbot_base" params="name">
     <link name="${name}_footprint">
@@ -115,6 +115,6 @@
         <!--<mesh filename="package://youbot_description/meshes/youbot_base/youbot_wheel.stl" />-->
         <geometry>
-          <sphere radius="${wheel_radius}"/>
-        </geometry>
+          				<mesh filename="package://youbot_description/meshes/youbot_base/wheel2.dae" />
+	</geometry>
         <material name="Orange"/>
       </visual>
@@ -160,8 +160,8 @@
       <visual>
         <origin xyz="0 0 0" rpy="0 0 0"/>
-        <geometry>
           <!--<mesh filename="package://youbot_description/meshes/youbot_base/youbot_wheel.stl" />-->
-          <sphere radius="${wheel_radius}"/>
-        </geometry>
+	<geometry>
+          				<mesh filename="package://youbot_description/meshes/youbot_base/wheel2.dae" />
+	</geometry>
         <material name="Orange"/>
       </visual>
@@ -209,7 +209,6 @@
         <origin xyz="0 0 0" rpy="0 0 0"/>
         <geometry>
-          <!--<mesh filename="package://youbot_description/meshes/youbot_base/youbot_wheel.stl" />-->
-          <sphere radius="${wheel_radius}"/>
-        </geometry>
+          				<mesh filename="package://youbot_description/meshes/youbot_base/wheel2.dae" />
+	</geometry>
         <material name="Orange"/>
       </visual>
@@ -255,8 +254,7 @@
       <visual>
         <origin xyz="0 0 0" rpy="0 0 0"/>
-        <geometry>
-          <!--<mesh filename="package://youbot_description/meshes/youbot_base/youbot_wheel.stl" />-->
-          <sphere radius="${wheel_radius}"/>
-        </geometry>
+       <geometry>
+          				<mesh filename="package://youbot_description/meshes/youbot_base/wheel2.dae" />
+	</geometry>
         <material name="Orange"/>
       </visual>
